Commit message: Working version update MBAC, BAC. Experiment on Block insertion complete

File: pyPack/bullet3/examples/pybullet/gym/pybullet_data/block3D.urdf (robot description, URDF)
Before this commit: robot block3D, 4 links, 3 joints
Links:
- link block: mass 2 -> 0.5; geometry collision box size=0.15 0.15 0.15; visual box size=0.15 0.15 0.15
Joints:
- joint slide_x: limit lower=-10.0 upper=10.0 effort=1000.0 velocity=5.0 -> lower=-15.0 upper=15.0 effort=1000.0 velocity=5.0
- joint slide_y: limit lower=-10.0 upper=10.0 effort=1000.0 velocity=5.0 -> lower=-15.0 upper=15.0 effort=1000.0 velocity=5.0
- joint slide_z: limit lower=-10.0 upper=10.0 effort=1000.0 velocity=5.0 -> lower=-15.0 upper=15.0 effort=1000.0 velocity=5.0

File: pyPack/bullet3/examples/pybullet/gym/pybullet_data/block_insert_fl3.urdf (robot description, URDF)
Before this commit: robot slot3, 2 links, 1 joints
Joints:
- removed joint base_fl1
- added joint base_fl3: type fixed, parent plane, child fl3, origin xyz=0.1 0.5 0.05
