Commit message: Fixed bug of segment state collection, added modified approach to IS

File: pyPack/bullet3/examples/pybullet/gym/pybullet_data/blockSlide2D.urdf (robot description, URDF)
Before this commit: robot block, 3 links, 2 joints
Links:
- link block: mass 0.5 -> 0.25; geometry collision box size=0.3 0.3 0.3; visual box size=0.3 0.3 0.3
Joints:
- joint slide_x: origin xyz=0.0 0.0 0.075 -> xyz=0.0 0.0 0.15

File: pyPack/bullet3/examples/pybullet/gym/pybullet_data/block_slide_w1.urdf (robot description, URDF)
Before this commit: robot wall1, 2 links, 1 joints
Links:
- link wl1: geometry collision box size=0.05 2 2; visual box size=0.05 2 2
Joints:
- joint base_wl1: origin xyz=-0.025 0.5 0.5 -> xyz=-0.025 1 1

File: pyPack/bullet3/examples/pybullet/gym/pybullet_data/block_slide_w2.urdf (robot description, URDF)
Before this commit: robot wall2, 2 links, 1 joints
Links:
- link wl2: geometry collision box size=2 0.05 2; visual box size=2 0.05 2
Joints:
- joint base_wl2: origin xyz=0.5 -0.025 0.5 -> xyz=1 -0.025 1

File: pyPack/bullet3/examples/pybullet/gym/pybullet_data/block_slide_w3.urdf (robot description, URDF)
Before this commit: robot wall3, 2 links, 1 joints
Links:
- link wl3: geometry collision box size=2 2 0.05; visual box size=2 2 0.05
Joints:
- joint base_wl3: origin xyz=0.5 0.5 -0.025 -> xyz=1 1 -0.025
