Commit message: Updated environments for experimental evaluation

File: pyPack/bullet3/examples/pybullet/gym/pybullet_data/block.urdf (robot description, URDF)
Before this commit: robot block, 3 links, 2 joints
Links:
- link block: geometry collision box size=0.1 0.096 0.1; visual box size=0.1 0.096 0.1

File: pyPack/bullet3/examples/pybullet/gym/pybullet_data/block3D.urdf (robot description, URDF)
Before this commit: robot block3D, 4 links, 3 joints
Links:
- link block: geometry collision box size=0.3 0.3 0.3; visual box size=0.3 0.3 0.3

File: pyPack/bullet3/examples/pybullet/gym/pybullet_data/block_insert_flm1.urdf (robot description, URDF)
Before this commit: robot wall1, 2 links, 1 joints
Links:
- removed link wl1
- added link fl1, mass 2.0; collision box size=0.1 0.18 0.1; visual box size=0.1 0.18 0.1
Joints:
- removed joint base_wl1
- added joint base_fl1: type fixed, parent plane, child fl1, origin xyz=0.0 0.66 0.05

File: pyPack/bullet3/examples/pybullet/gym/pybullet_data/block_insert_flm2.urdf (robot description, URDF)
Before this commit: robot wall1, 2 links, 1 joints
Links:
- removed link wl1
- added link fl2, mass 2.0; collision box size=0.1 0.22 0.1; visual box size=0.1 0.22 0.1
Joints:
- removed joint base_wl1
- added joint base_fl2: type fixed, parent plane, child fl2, origin xyz=0.0 0.36 0.05

File: pyPack/bullet3/examples/pybullet/gym/pybullet_data/block_slide_w1.urdf (robot description, URDF)
Before this commit: robot wall1, 2 links, 1 joints
Links:
- removed link wl1
- added link wl2, mass 3.0; collision box size=1.5 0.05 0.5; visual box size=1.5 0.05 0.5
Joints:
- removed joint base_wl1
- added joint base_wl2: type fixed, parent plane, child wl2, origin xyz=0.75 -0.025 0.25

File: pyPack/bullet3/examples/pybullet/gym/pybullet_data/block_slide_w3.urdf (robot description, URDF)
Before this commit: robot wall3, 2 links, 1 joints
Links:
- removed link wl3
- added link fl1, mass 1.5; collision box size=1.5 1.5 0.05; visual box size=1.5 1.5 0.05
Joints:
- removed joint base_wl3
- added joint base_fl: type fixed, parent plane, child fl1, origin xyz=0.75 0.75 -0.025

Commit message: Working configuration of Block Insertion, 85% success rate 90% similarity

File: pyPack/bullet3/examples/pybullet/gym/pybullet_data/block.urdf (robot description, URDF)
Before this commit: robot block, 3 links, 2 joints
Links:
- link block: geometry collision box size=0.1 0.095 0.1; visual box size=0.1 0.095 0.1

File: pyPack/bullet3/examples/pybullet/gym/pybullet_data/block3D.urdf (robot description, URDF)
Before this commit: robot block3D, 4 links, 3 joints
Joints:
- joint slide_x: limit lower=-15.0 upper=15.0 effort=1000.0 velocity=5.0 -> lower=-10.0 upper=10.0 effort=1000.0 velocity=5.0
- joint slide_y: limit lower=-15.0 upper=15.0 effort=1000.0 velocity=5.0 -> lower=-10.0 upper=10.0 effort=1000.0 velocity=5.0
- joint slide_z: limit lower=-15.0 upper=15.0 effort=1000.0 velocity=5.0 -> lower=-10.0 upper=10.0 effort=1000.0 velocity=5.0

Commit message: Cleaned IOAC

File: pyPack/bullet3/examples/pybullet/gym/pybullet_data/block.urdf (robot description, URDF)
Before this commit: robot block, 3 links, 2 joints
Links:
- link block: mass 2 -> 0.5
